File: hardware/board/harp_core_rp2040_w_isolated_usb.kicad_sch (KiCad schematic)
At the start: 49 parts, among them J1 Conn_01x03_Male, J2 AudioJack3, J5 USB_C_Receptacle_USB2.0, U2 TPD2EUSB30, U3 ADUM4160, U4 RP2040, U5 W25Q16JVUXIQ, X1 ECS-TXO-2016

Commit message: add tvs diodes to inputs
Parts:
- J1: now not fitted
Changed lines of the file:
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@@
 	(label "QSPI_CLK"
 		(at 172.085 90.805 180)
-		(fields_autoplaced yes)
 		(effects
 			(font
@@
 	(label "QSPI_CS"
 		(at 172.085 75.565 180)
-		(fields_autoplaced yes)
 		(effects
 			(font
@@
 	(label "HARP_CLK_SYNC"
 		(at 242.57 86.995 0)
-		(fields_autoplaced yes)
 		(effects
 			(font
@@
 	(label "VDD1"
 		(at 120.65 32.385 180)
-		(fields_autoplaced yes)
 		(effects
 			(font
@@
 	(label "USB_Boot"
 		(at 31.115 102.235 0)
-		(fields_autoplaced yes)
 		(effects
 			(font
@@
 	(label "D-"
 		(at 110.49 42.545 180)
-		(fields_autoplaced yes)
 		(effects
 			(font
@@
 	(label "QSPI_CS"
 		(at 52.705 102.235 0)
-		(fields_autoplaced yes)
 		(effects
 			(font
@@
 	(label "QSPI_D2"
 		(at 271.145 38.1 0)
-		(fields_autoplaced yes)
 		(effects
 			(font
@@
 	(label "UART0_RXD"
 		(at 24.765 88.265 0)
-		(fields_autoplaced yes)
 		(effects
 			(font
@@
 	(label "VDD1"
 		(at 38.735 139.065 180)
-		(fields_autoplaced yes)
 		(effects
 			(font
@@
 	(label "HARP_CLK_SYNC"
 		(at 40.005 122.555 0)
-		(fields_autoplaced yes)
 		(effects
 			(font
@@
 	(label "QSPI_D3"
 		(at 172.085 86.995 180)
-		(fields_autoplaced yes)
 		(effects
 			(font
@@
 	(label "UART0_TXD"
 		(at 241.935 74.295 0)
-		(fields_autoplaced yes)
 		(effects
 			(font
@@
 	(label "DD+"
 		(at 161.29 40.005 0)
-		(fields_autoplaced yes)
 		(effects
 			(font
@@
 	(label "QSPI_D3"
 		(at 271.145 40.64 0)
-		(fields_autoplaced yes)
 		(effects
 			(font
@@
 	(label "DD+"
 		(at 249.555 64.135 0)
-		(fields_autoplaced yes)
 		(effects
 			(font
@@
 	(label "D-"
 		(at 69.85 38.1 0)
-		(fields_autoplaced yes)
 		(effects
 			(font
@@
 	(label "DD-"
 		(at 249.555 66.675 0)
-		(fields_autoplaced yes)
 		(effects
 			(font
@@
 	(label "QSPI_D2"
 		(at 172.085 84.455 180)
-		(fields_autoplaced yes)
 		(effects
 			(font
@@
 	(label "QSPI_D0"
 		(at 172.085 79.375 180)
-		(fields_autoplaced yes)
 		(effects
 			(font
@@
 	(label "QSPI_D1"
 		(at 172.085 81.915 180)
-		(fields_autoplaced yes)
 		(effects
 			(font
@@
 	(label "QSPI_CLK"
 		(at 241.935 38.1 180)
-		(fields_autoplaced yes)
 		(effects
 			(font
@@
 	(label "DD-"
 		(at 161.29 42.545 0)
-		(fields_autoplaced yes)
 		(effects
 			(font
@@
 	(label "D+"
 		(at 110.49 40.005 180)
-		(fields_autoplaced yes)
 		(effects
 			(font
@@
 	(label "QSPI_CS"
 		(at 241.935 33.02 180)
-		(fields_autoplaced yes)
 		(effects
 			(font
@@
 	(label "QSPI_D1"
 		(at 271.145 33.02 0)
-		(fields_autoplaced yes)
 		(effects
 			(font
@@
 	(label "D+"
 		(at 69.85 43.18 0)
-		(fields_autoplaced yes)
 		(effects
 			(font
@@
 	(label "QSPI_D0"
 		(at 271.145 30.48 0)
-		(fields_autoplaced yes)
 		(effects
 			(font
@@
 	(label "UART0_RXD"
 		(at 241.935 76.835 0)
-		(fields_autoplaced yes)
 		(effects
 			(font
@@
 	(label "UART0_TXD"
 		(at 24.765 85.725 0)
-		(fields_autoplaced yes)
 		(effects
 			(font
@@
 		(shape input)
 		(at 241.935 130.175 0)
-		(fields_autoplaced yes)
 		(effects
 			(font
@@
 		(shape input)
 		(at 241.935 120.015 0)
-		(fields_autoplaced yes)
 		(effects
 			(font
@@
 		(shape input)
 		(at 241.935 122.555 0)
-		(fields_autoplaced yes)
 		(effects
 			(font
@@
 		(shape input)
 		(at 241.935 99.695 0)
-		(fields_autoplaced yes)
 		(effects
 			(font
@@
 		(shape input)
 		(at 241.935 102.235 0)
-		(fields_autoplaced yes)
 		(effects
 			(font
@@
 		(shape input)
 		(at 241.935 114.935 0)
-		(fields_autoplaced yes)
 		(effects
 			(font
@@
 		(shape input)
 		(at 241.935 117.475 0)
-		(fields_autoplaced yes)
 		(effects
 			(font
@@
 		(shape input)
 		(at 241.935 97.155 0)
-		(fields_autoplaced yes)
 		(effects
 			(font
@@
 		(shape input)
 		(at 241.935 132.715 0)
-		(fields_autoplaced yes)
 		(effects
 			(font
@@
 		(shape input)
 		(at 241.935 127.635 0)
-		(fields_autoplaced yes)
 		(effects
 			(font
@@
 		(shape input)
 		(at 241.935 125.095 0)
-		(fields_autoplaced yes)
 		(effects
 			(font
@@
 		(in_bom yes)
 		(on_board yes)
-		(dnp no)
+		(dnp yes)
 		(property "Reference" "J1"
 			(at 17.145 84.455 0)
