File: hardware/board/harp_treadmill.kicad_sch (KiCad schematic)
At the start: 1 part

Commit message: add tvs diodes to inputs
Other:
- company: (none) -> The Allen Institute
- title: (none) -> harp.device.treadmill-driver
Changed lines of the file:
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@@
 	(generator_version "8.0")
 	(paper "A4")
+	(title_block
+		(title "harp.device.treadmill-driver")
+		(date "2025-09-08")
+		(rev "1.3.0")
+		(company "The Allen Institute")
+	)
 	(wire
 		(pts
