File: hardware/board/power_supplies.kicad_sch (KiCad schematic)
At the start: 43 parts, among them J4 Barrel_Jack_Switch, U13 LM27762, U2 LP2985-3.3, U6 REF2033, U8 LT3506

Commit message: add tvs diodes to inputs
Parts:
- C38: Manufacturer (none) -> Samsung Electro-Mechanics; PCBWay Link todo -> (none)
Changed lines of the file:
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@@
 			)
 		)
-		(property "PCBWay Link" "todo"
+		(property "Manufacturer" "Samsung Electro-Mechanics"
 			(at 107.315 118.745 0)
 			(effects
